Commit message: integrated SLAM & odometry with the Main scene

File: Assets/Urdf/default/unity_boat.urdf (robot description, URDF)
Before this commit: robot unity_boat, 6 links, 5 joints
Links:
- link boat_rear: mass None -> 1
- link engine: mass None -> 1
- link left_balancer: mass None -> 1
- link right_balancer: mass None -> 1
- link video_camera: mass None -> 1
Joints:
- removed joint base_link_boat_rear_joint
- removed joint base_link_left_balancer_joint
- removed joint base_link_right_balancer_joint
- removed joint base_link_video_camera_joint
- removed joint boat_rear_engine_joint
- added joint base_to_boat_rear: type fixed, parent base_link, child boat_rear, origin xyz=-0.8 0 0
- added joint base_to_left_balancer: type fixed, parent base_link, child left_balancer, origin xyz=0.7 0.3 0
- added joint base_to_right_balancer: type fixed, parent base_link, child right_balancer, origin xyz=0.7 -0.3 0
- added joint base_to_video_camera: type fixed, parent base_link, child video_camera, origin xyz=0.4 0 0.325
- added joint rear_to_engine: type revolute, parent boat_rear, child engine, origin xyz=-0.35 0 0, axis 0 0 1, limit lower=-0.4 upper=0.4 effort=1000 velocity=1000
